File: stamp/battery-protection.sch (KiCad schematic (older format))
At the start: 5 parts

Commit message: Pre-review
Parts:
- C5: renamed from C?; value C -> 100nF; footprint Capacitor_SMD:C_0402_1005Metric -> Capacitor_SMD:C_0603_1608Metric
- gave numbers to parts that had none: 4
Other:
- note removed: "TODO: Resistor/Cap Values"
Changed lines of the file:
@@
 AP9101CK6-ADTRG1
 $Comp
-L power:GND #PWR?
+L power:GND #PWR0110
 U 1 1 5FC96E83
 P 3800 3200
-F 0 "#PWR?" H 3800 2950 50  0001 C CNN
+F 0 "#PWR0110" H 3800 2950 50  0001 C CNN
 F 1 "GND" H 3805 3027 50  0000 C CNN
 F 2 "" H 3800 3200 50  0001 C CNN
@@
 $EndComp
 $Comp
-L Device:C C?
-U 1 1 5FC96E89
-P 4950 2750
-F 0 "C?" H 5065 2796 50  0000 L CNN
-F 1 "C" H 5065 2705 50  0000 L CNN
-F 2 "Capacitor_SMD:C_0402_1005Metric" H 4988 2600 50  0001 C CNN
-F 3 "~" H 4950 2750 50  0001 C CNN
-	1    4950 2750
-	1    0    0    -1
-$EndComp
-$Comp
-L Device:R R?
+L Device:R R6
 U 1 1 5FC96E8F
 P 5100 3450
-F 0 "R?" H 5170 3496 50  0000 L CNN
+F 0 "R6" H 5170 3496 50  0000 L CNN
 F 1 "2.7kOhm" H 5170 3405 50  0000 L CNN
 F 2 "Resistor_SMD:R_0402_1005Metric" V 5030 3450 50  0001 C CNN
@@
 $EndComp
 $Comp
-L Device:R R?
+L Device:R R5
 U 1 1 5FC96E95
 P 4700 2600
-F 0 "R?" V 4800 2600 50  0000 C CNN
+F 0 "R5" V 4800 2600 50  0000 C CNN
 F 1 "330" V 4700 2600 50  0000 C CNN
 F 2 "Resistor_SMD:R_0402_1005Metric" V 4630 2600 50  0001 C CNN
@@
 Wire Wire Line
 	5100 2900 5100 3300
-Text Notes 3850 2250 0    50   ~ 0
+Text Notes 7350 7500 0    50   ~ 0
 Battery Protection
-Text Notes 3850 4650 0    50   ~ 0
-TODO: Resistor/Cap Values
-Wire Notes Line
-	7250 2150 7250 4700
 Connection ~ 4950 2600
 Wire Wire Line
@@
 	4950 3200 4950 4000
 $Comp
-L Everything:FS8205 U?
+L Everything:FS8205 U3
 U 1 1 5FC96EAA
 P 6750 3150
-F 0 "U?" H 6750 3265 50  0000 C CNN
+F 0 "U3" H 6750 3265 50  0000 C CNN
 F 1 "FS8205" H 6750 3174 50  0000 C CNN
 F 2 "Package_TO_SOT_SMD:SOT-23-6" H 6750 3150 50  0001 C CNN
@@
 Wire Wire Line
 	6400 2900 6450 2900
-Wire Notes Line
-	3450 2150 3450 4700
-Wire Notes Line
-	3450 4700 7250 4700
-Wire Notes Line
-	3450 2150 7250 2150
 Wire Wire Line
 	4600 3200 4600 3600
@@
 	6100 3000 6450 3000
 $Comp
-L Battery_Management:AP9101CK6 U?
+L Battery_Management:AP9101CK6 U2
 U 1 1 5FC96EC8
 P 5700 2900
-F 0 "U?" H 5700 3381 50  0000 C CNN
+F 0 "U2" H 5700 3381 50  0000 C CNN
 F 1 "AP9101CK6" H 5700 3290 50  0000 C CNN
 F 2 "Package_TO_SOT_SMD:SOT-23-6" H 5700 2900 50  0001 C CNN
@@
 -BATT
 $Comp
-L power:GND #PWR?
+L power:GND #PWR0111
 U 1 1 5FC97A6C
 P 1200 850
-F 0 "#PWR?" H 1200 600 50  0001 C CNN
+F 0 "#PWR0111" H 1200 600 50  0001 C CNN
 F 1 "GND" H 1205 677 50  0000 C CNN
 F 2 "" H 1200 850 50  0001 C CNN
@@
 Wire Wire Line
 	900  850  1200 850
+$Comp
+L Device:C C5
+U 1 1 5FC96E89
+P 4950 2750
+F 0 "C5" H 5065 2796 50  0000 L CNN
+F 1 "100nF" H 5065 2705 50  0000 L CNN
+F 2 "Capacitor_SMD:C_0603_1608Metric" H 4988 2600 50  0001 C CNN
+F 3 "~" H 4950 2750 50  0001 C CNN
+	1    4950 2750
+	1    0    0    -1
+$EndComp
 $EndSCHEMATC

Commit message: Update components, regenerate output
Parts:
- R6: footprint Resistor_SMD:R_0402_1005Metric -> Resistor_SMD:R_0603_1608Metric
Changed lines of the file:
@@
 F 0 "R6" H 5170 3496 50  0000 L CNN
 F 1 "2.7kOhm" H 5170 3405 50  0000 L CNN
-F 2 "Resistor_SMD:R_0402_1005Metric" V 5030 3450 50  0001 C CNN
+F 2 "Resistor_SMD:R_0603_1608Metric" V 5030 3450 50  0001 C CNN
 F 3 "~" H 5100 3450 50  0001 C CNN
 	1    5100 3450
