File: stamp/power-path.sch (KiCad schematic (older format))
At the start: 3 parts

Commit message: Pre-review
Parts:
- gave numbers to parts that had none: 3
Changed lines of the file:
@@
 Power Path (VMAX selection)
 $Comp
-L power:GND #PWR?
+L power:GND #PWR0105
 U 1 1 5FC78D8B
 P 5450 3650
-F 0 "#PWR?" H 5450 3400 50  0001 C CNN
+F 0 "#PWR0105" H 5450 3400 50  0001 C CNN
 F 1 "GND" H 5455 3477 50  0000 C CNN
 F 2 "" H 5450 3650 50  0001 C CNN
@@
 VMAX
 $Comp
-L Device:D_Schottky D?
+L Device:D_Schottky D4
 U 1 1 5FC78D94
 P 4900 3450
-F 0 "D?" H 4900 3233 50  0000 C CNN
+F 0 "D4" H 4900 3233 50  0000 C CNN
 F 1 "D_Schottky" H 4900 3324 50  0000 C CNN
 F 2 "Diode_SMD:D_SOD-123" H 4900 3450 50  0001 C CNN
@@
 	4600 3450 4750 3450
 $Comp
-L Device:R R?
+L Device:R R4
 U 1 1 5FC78D9B
 P 5050 3650
-F 0 "R?" V 5000 3800 50  0000 C CNN
+F 0 "R4" V 5000 3800 50  0000 C CNN
 F 1 "100K" V 5050 3650 50  0000 C CNN
 F 2 "Resistor_SMD:R_0402_1005Metric" V 4980 3650 50  0001 C CNN
@@
 	5200 3650 5450 3650
 $Comp
-L Device:Q_PMOS_GSD Q?
+L Device:Q_PMOS_GSD Q1
 U 1 1 5FC78DA4
 P 4950 3000
-F 0 "Q?" H 5155 3046 50  0000 L CNN
+F 0 "Q1" H 5155 3046 50  0000 L CNN
 F 1 "Q_PMOS_GSD" H 5155 2955 50  0000 L CNN
 F 2 "Package_TO_SOT_SMD:SOT-23" H 5150 3100 50  0001 C CNN
@@
 GND
 $Comp
-L power:GND #PWR?
+L power:GND #PWR0106
 U 1 1 5FC7A866
 P 1100 950
-F 0 "#PWR?" H 1100 700 50  0001 C CNN
+F 0 "#PWR0106" H 1100 700 50  0001 C CNN
 F 1 "GND" H 1105 777 50  0000 C CNN
 F 2 "" H 1100 950 50  0001 C CNN

Commit message: Add fabrication outputs, not jlc corrected yet
Parts:
- Q1: value Q_PMOS_GSD -> SI2301CDS-T1-GE3
Other:
- note added: "D"
- note added: "G"
- note added: "S"
Changed lines of the file:
@@
 P 4950 3000
 F 0 "Q1" H 5155 3046 50  0000 L CNN
-F 1 "Q_PMOS_GSD" H 5155 2955 50  0000 L CNN
+F 1 "SI2301CDS-T1-GE3" H 5155 2955 50  0000 L CNN
 F 2 "Package_TO_SOT_SMD:SOT-23" H 5150 3100 50  0001 C CNN
 F 3 "~" H 4950 3000 50  0001 C CNN
@@
 Wire Wire Line
 	900  950  1100 950
+Text Notes 4950 2850 0    50   ~ 0
+D
+Text Notes 4950 3200 0    50   ~ 0
+S
+Text Notes 4800 3000 0    50   ~ 0
+G
 $EndSCHEMATC

Commit message: Update exports/screenshots
Parts:
- D4: value D_Schottky -> B5819W
Changed lines of the file:
@@
 P 4900 3450
 F 0 "D4" H 4900 3233 50  0000 C CNN
-F 1 "D_Schottky" H 4900 3324 50  0000 C CNN
+F 1 "B5819W" H 4900 3324 50  0000 C CNN
 F 2 "Diode_SMD:D_SOD-123" H 4900 3450 50  0001 C CNN
 F 3 "~" H 4900 3450 50  0001 C CNN
