File: stamp/lipo-stamp-proto.sch (KiCad schematic (older format))
At the start: 11 parts

Commit message: Pre-review
Parts:
- added R1: 2.2K, Resistor_SMD:R_0402_1005Metric, symbol Device:R
- F1: value Polyfuse -> 2A Polyfuse
- renumbered TP8 to TP5, TP5 to TP6, TP6 to TP7, TP7 to TP8
Connections:
- net GND: now also R1.2
- net charge-controller/PROG: now also R1.1
- net 3V3_OUT renamed +3v3
- net 3V3_REG_EN renamed 3v3_EN
- net STAT_OUT renamed STAT
- net VMAX_OUT renamed VMAX
- no-connect marks 0 -> 1
Other:
- note added: "* See comment on 3v3 reg re: max current\nTBD: Actual max current threshold, right now\n100mA is a conservative guess"
- note added: "+3v3 Regulator when\n3v3_EN is high, otherwise\ndisabled.\n\n* Regulator supports 600mA\noutput, but we probably don't\nhave thermals for that"
- note added: "+3v3: 3.3v, 100mA max*"
- note added: "2.2K is roughly 500mA"
- note added: "2020-11-29"
- note added: "2A polyfuse disconnects\n-BATT_RAW when total\ncontinuous current is\n>= 2A"
- note added: "Battery Negative"
- note added: "Battery Positive"
- note added: "Battery Protection will\ndisconnect -BATT from GND\nwhen voltage is too high/low,\notherwise connect -BATT\nto GND (output)"
- note added: "Constant Current Charge\nController with 500mA max\ncharge current"
- note added: "GREEN LED"
- note added: "INPUTS"
- note added: "LEDs"
- note added: "LiPo Stamp v0.3.0"
- note added: "Low: Charging, High: Not Charging"
- note added: "Low: Disable 3v3 Reg, High: Enable 3v3 Reg"
- note added: "OUTPUTS"
- note added: "On: Charging, Off: Not Charging"
- note added: "On: Standby, Off: Charging or no power"
- note added: "Power path switches VMAX to\n+CHARGE when present,\notherwise +BATT"
- note added: "RED LED"
- note added: "STAGE 1: 2A Polyfuse"
- note added: "STAGE 2: Battery Protection"
- note added: "STAGE 3: Battery Charge Controller"
- note added: "STAGE 4: Power Path Selection"
- note added: "STAGE 5: +3v3 Regulator"
- note added: "Total current for all outputs is 2A when battery powered.\nTotal current for +CHARGE is 1A, 0.5A to charge, 0.5A to VMAX\nALWAYS use GND output, NOT -BATT, to maintain protection"
- note added: "USB/+5v0 Input"
- note added: "USB/GND Input"
- note added: "VBAT: 3.0-4.2v, 2A max"
- note added: "VMAX: 3.0-4.8v, 500mA max"
- note removed: "+2v5 ..= +4v2"
- note removed: "+2v5 ..= +5v5"
- note removed: "+3v3 Regulated Output"
- note removed: "+3v3 Regulation EN (disable low)"
- note removed: "0v0 OR +3v3"
- note removed: "0v0 OR +5v5"
- note removed: "2A"
- note removed: "2A Polyfuse"
- note removed: "500mA"
- note removed: "500mA ..= 1A"
- note removed: "500mA ..= 2A"
- note removed: "Charge Status Out"
- note removed: "Current In/Out"
- note removed: "Logical GND"
- note removed: "Negative Battery Terminal"
- note removed: "Negative USB Supply"
- note removed: "Positive Battery, Source Limited"
- note removed: "Positive USB Supply"
- note removed: "Postive Battery Terminal"
- note removed: "Voltage In/Out"
- note removed: "max(+BATT, +CHARGE)"
- moved on the sheet: F1, TP1, TP10, TP2, TP3, TP4, TP5, TP6, TP7, TP8, TP9

Commit message: Update exports/screenshots
Parts:
- F1: value 2A Polyfuse -> nSMD200
Changed lines of the file:
@@
 P 1550 4000
 F 0 "F1" V 1325 4000 50  0000 C CNN
-F 1 "2A Polyfuse" V 1416 4000 50  0000 C CNN
+F 1 "nSMD200" V 1416 4000 50  0000 C CNN
 F 2 "Fuse:Fuse_1206_3216Metric_Castellated" H 1600 3800 50  0001 L CNN
 F 3 "~" H 1550 4000 50  0001 C CNN

Commit message: Add more filter caps
Parts:
- added C7: 1uF, Capacitor_SMD:C_0603_1608Metric, symbol Device:C
Connections:
- net +CHARGE: now also C7.1
- net GND: now also C7.2
Other:
- note added: "Input filter for noisy switching supplies"
Changed lines of the file:
@@
 Wire Notes Line
 	2650 2050 2650 550
-Text Label 4900 3800 2    50   ~ 0
-+CHARGE
 Text Label 4900 3900 2    50   ~ 0
 +BATT
@@
 Text Notes 8400 3350 0    50   ~ 0
 STAGE 5: +3v3 Regulator
+$Comp
+L Device:C C?
+U 1 1 5FC542AF
+P 5050 2300
+AR Path="/5FC8E9A5/5FC542AF" Ref="C?"  Part="1"
+AR Path="/5FC542AF" Ref="C7"  Part="1"
+F 0 "C7" H 5165 2346 50  0000 L CNN
+F 1 "1uF" H 5165 2255 50  0000 L CNN
+F 2 "Capacitor_SMD:C_0603_1608Metric" H 5088 2150 50  0001 C CNN
+F 3 "~" H 5050 2300 50  0001 C CNN
+	1    5050 2300
+	1    0    0    -1
+$EndComp
+Text Label 4900 3800 2    50   ~ 0
++CHARGE
+Text Label 5050 2150 2    50   ~ 0
++CHARGE
+$Comp
+L power:GND #PWR0113
+U 1 1 5FC5C63A
+P 5050 2450
+F 0 "#PWR0113" H 5050 2200 50  0001 C CNN
+F 1 "GND" H 5055 2277 50  0000 C CNN
+F 2 "" H 5050 2450 50  0001 C CNN
+F 3 "" H 5050 2450 50  0001 C CNN
+	1    5050 2450
+	1    0    0    -1
+$EndComp
+Text Notes 5400 2350 0    50   ~ 0
+Input filter for noisy switching supplies
 $EndSCHEMATC
